File: kicad/Arducon.sch (KiCad schematic (older format))
At the start: 70 parts, among them J101 To Radio, J102 DB9 Female, J103 To Antenna, J104 Conn_01x08, J105 Conn_01x08, J106 Logic Level, J107 External Power Source, J108 Controlled Power, J109 Conn_01x01, J110 Conn_01x01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

Commit message: BOM Script Updates
o Schematic and script changes to improve BOM usefulness
Parts:
- D101, D102, D103, D105, D106, D107, D109, Q101, Q103, Q104, R105, R107, R108, R110, R112, RV101, U101, U102, U104: Description (none) -> TBD; Manufacturer (none) -> TBD; Manufacturer PN (none) -> TBD
- D104, Q102: Manufacturer (none) -> TBD; Manufacturer PN (none) -> TBD
Changed lines of the file:
@@
 F 4 "2195-RV-3028-C732.768KHZ1PPM-TA-QCCT-ND" H 7350 3450 50  0001 C CNN "Part No."
 F 5 "<a href=\"https://www.digikey.com/products/en?keywords=2195-RV-3028-C732.768KHZ1PPM-TA-QCCT-ND\">Link</a>" H 7350 3450 50  0001 C CNN "Link"
+F 6 "" H 7350 3450 50  0001 C CNN "Manufacturer"
+F 7 "" H 7350 3450 50  0001 C CNN "Manufacturer PN"
+F 8 "" H 7350 3450 50  0001 C CNN "Description"
 	1    7350 3450
 	1    0    0    -1
@@
 F 4 "TC33X-103ECT-ND" H 4300 2250 50  0001 C CNN "Part No."
 F 5 "<a href=\"https://www.digikey.com/products/en?keywords=TC33X-103ECT-ND\">Link</a>" H 4300 2250 50  0001 C CNN "Link"
+F 6 "TBD" H 4300 2250 50  0001 C CNN "Manufacturer"
+F 7 "TBD" H 4300 2250 50  0001 C CNN "Manufacturer PN"
+F 8 "TBD" H 4300 2250 50  0001 C CNN "Description"
 	1    4300 2250
 	-1   0    0    1
@@
 F 4 "311-162KCRCT-ND" H 2900 6250 50  0001 C CNN "Part No."
 F 5 "<a href=\"https://www.digikey.com/products/en?keywords=311-162KCRCT-ND\">Link</a>" H 2900 6250 50  0001 C CNN "Link"
+F 6 "TBD" V 2900 6250 50  0001 C CNN "Manufacturer"
+F 7 "TBD" V 2900 6250 50  0001 C CNN "Manufacturer PN"
+F 8 "TBD" V 2900 6250 50  0001 C CNN "Description"
 	1    2900 6250
 	0    1    1    0
@@
 F 4 "800-3576-ND" H 14100 2800 50  0001 C CNN "Part No."
 F 5 "<a href=\"https://www.digikey.com/products/en?keywords=800-3576-ND\">Link</a>" H 14100 2800 50  0001 C CNN "Link"
+F 6 "TBD" H 14100 2800 50  0001 C CNN "Manufacturer"
+F 7 "TBD" H 14100 2800 50  0001 C CNN "Manufacturer PN"
+F 8 "TBD" H 14100 2800 50  0001 C CNN "Description"
 	1    14100 2800
 	1    0    0    -1
@@
 F 4 "296-14529-1-ND" H 10350 3700 50  0001 C CNN "Part No."
 F 5 "<a href=\"https://www.digikey.com/products/en?keywords=296-14529-1-ND\">Link</a>" H 10350 3700 50  0001 C CNN "Link"
+F 6 "TBD" H 10350 3700 50  0001 C CNN "Manufacturer"
+F 7 "TBD" H 10350 3700 50  0001 C CNN "Manufacturer PN"
+F 8 "TBD" H 10350 3700 50  0001 C CNN "Description"
 	4    10350 3700
 	1    0    0    -1
@@
 F 4 "576-1281-1-ND " H 10350 1700 50  0001 C CNN "Part No."
 F 5 "<a href=\"https://www.digikey.com/products/en?keywords=576-1281-1-ND \">Link</a>" H 10350 1700 50  0001 C CNN "Link"
+F 6 "TBD" H 10350 1700 50  0001 C CNN "Manufacturer"
+F 7 "TBD" H 10350 1700 50  0001 C CNN "Manufacturer PN"
+F 8 "TBD" H 10350 1700 50  0001 C CNN "Description"
 	1    10350 1700
 	1    0    0    -1
@@
 F 4 "LMN400E01DICT-ND" H 13550 7600 50  0001 C CNN "Part No."
 F 5 "<a href=\"https://www.digikey.com/products/en?keywords=LMN400E01DICT-ND\">Link</a>" H 13550 7600 50  0001 C CNN "Link"
+F 6 "TBD" H 13550 7600 50  0001 C CNN "Manufacturer"
+F 7 "TBD" H 13550 7600 50  0001 C CNN "Manufacturer PN"
+F 8 "" H 13550 7600 50  0001 C CNN "Description"
 	1    13550 7600
 	1    0    0    -1
@@
 F 4 "RMCF0805FT1M00CT-ND" H 3100 4550 60  0001 C CNN "Part No."
 F 5 "<a href=\"https://www.digikey.com/products/en?keywords=RMCF0805FT1M00CT-ND\">Link</a>" H 3100 4550 60  0001 C CNN "Link"
+F 6 "TBD" V 3100 4550 50  0001 C CNN "Manufacturer"
+F 7 "TBD" V 3100 4550 50  0001 C CNN "Manufacturer PN"
+F 8 "TBD" V 3100 4550 50  0001 C CNN "Description"
 	1    3100 4550
 	1    0    0    -1
@@
 F 4 "MSS1P4-M3/89AGICT-ND" H 3700 7100 50  0001 C CNN "Part No."
 F 5 "<a href=\"https://www.digikey.com/products/en?keywords=MSS1P4-M3/89AGICT-ND\">Link</a>" H 3700 7100 50  0001 C CNN "Link"
+F 6 "TBD" H 3700 7100 50  0001 C CNN "Manufacturer"
+F 7 "TBD" H 3700 7100 50  0001 C CNN "Manufacturer PN"
+F 8 "TBD" H 3700 7100 50  0001 C CNN "Description"
 	1    3700 7100
 	-1   0    0    -1
@@
 F 4 "CG0603MLC-05LECT-ND" H 2150 8200 50  0001 C CNN "Part No."
 F 5 "<a href=\"https://www.digikey.com/products/en?keywords=CG0603MLC-05LECT-ND\">Link</a>" H 2150 8200 50  0001 C CNN "Link"
+F 6 "TBD" H 2150 8200 50  0001 C CNN "Manufacturer"
+F 7 "TBD" H 2150 8200 50  0001 C CNN "Manufacturer PN"
+F 8 "TBD" H 2150 8200 50  0001 C CNN "Description"
 	1    2150 8200
 	0    -1   -1   0
@@
 F 4 "CG0603MLC-05LECT-ND" H 2400 8200 50  0001 C CNN "Part No."
 F 5 "<a href=\"https://www.digikey.com/products/en?keywords=CG0603MLC-05LECT-ND\">Link</a>" H 2400 8200 50  0001 C CNN "Link"
+F 6 "TBD" H 2400 8200 50  0001 C CNN "Manufacturer"
+F 7 "TBD" H 2400 8200 50  0001 C CNN "Manufacturer PN"
+F 8 "" H 2400 8200 50  0001 C CNN "Description"
 	1    2400 8200
 	0    -1   -1   0
@@
 F 4 "CG0603MLC-05LECT-ND" H 2650 8200 50  0001 C CNN "Part No."
 F 5 "<a href=\"https://www.digikey.com/products/en?keywords=CG0603MLC-05LECT-ND\">Link</a>" H 2650 8200 50  0001 C CNN "Link"
+F 6 "TBD" H 2650 8200 50  0001 C CNN "Manufacturer"
+F 7 "TBD" H 2650 8200 50  0001 C CNN "Manufacturer PN"
+F 8 "TBD" H 2650 8200 50  0001 C CNN "Description"
 	1    2650 8200
 	0    -1   -1   0
@@
 F 4 "CG0603MLC-05LECT-ND" H 2900 8200 50  0001 C CNN "Part No."
 F 5 "<a href=\"https://www.digikey.com/products/en?keywords=CG0603MLC-05LECT-ND\">Link</a>" H 2900 8200 50  0001 C CNN "Link"
+F 6 "TBD" H 2900 8200 50  0001 C CNN "Manufacturer"
+F 7 "TBD" H 2900 8200 50  0001 C CNN "Manufacturer PN"
+F 8 "TBD" H 2900 8200 50  0001 C CNN "Description"
 	1    2900 8200
 	0    -1   -1   0
@@
 F 4 "CG0603MLC-05LECT-ND" H 3150 8200 50  0001 C CNN "Part No."
 F 5 "<a href=\"https://www.digikey.com/products/en?keywords=CG0603MLC-05LECT-ND\">Link</a>" H 3150 8200 50  0001 C CNN "Link"
+F 6 "TBD" H 3150 8200 50  0001 C CNN "Manufacturer"
+F 7 "TBD" H 3150 8200 50  0001 C CNN "Manufacturer PN"
+F 8 "TBD" H 3150 8200 50  0001 C CNN "Description"
 	1    3150 8200
 	0    -1   -1   0
@@
 F 4 "311-10.0CRCT-ND" H 7150 6500 60  0001 C CNN "Part No."
 F 5 "<a href=\"https://www.digikey.com/products/en?keywords=311-10.0CRCT-ND\">Link</a>" H 7150 6500 60  0001 C CNN "Link"
+F 6 "TBD" V 7150 6500 50  0001 C CNN "Manufacturer"
+F 7 "TBD" V 7150 6500 50  0001 C CNN "Manufacturer PN"
+F 8 "TBD" V 7150 6500 50  0001 C CNN "Description"
 	1    7150 6500
 	0    -1   1    0
@@
 F 4 "311-10.0KCRCT-ND" H 3550 6450 60  0001 C CNN "Part No."
 F 5 "<a href=\"https://www.digikey.com/products/en?keywords=311-10.0KCRCT-ND\">Link</a>" H 3550 6450 60  0001 C CNN "Link"
+F 6 "TBD" V 3550 6450 50  0001 C CNN "Manufacturer"
+F 7 "TBD" V 3550 6450 50  0001 C CNN "Manufacturer PN"
+F 8 "TBD" V 3550 6450 50  0001 C CNN "Description"
 	1    3550 6450
 	-1   0    0    1
@@
 F 4 "MMBT2222ATPMSCT-ND" H 4100 3400 50  0001 C CNN "Part No."
 F 5 "<a href=\"https://www.digikey.com/products/en?keywords=MMBT2222ATPMSCT-ND\">Link</a>" H 4100 3400 50  0001 C CNN "Link"
-F 6 "" H 4100 3400 50  0001 C CNN "Manufacturer"
-F 7 "" H 4100 3400 50  0001 C CNN "Manufacturer PN"
-F 8 "" H 4100 3400 50  0001 C CNN "Description"
+F 6 "TBD" H 4100 3400 50  0001 C CNN "Manufacturer"
+F 7 "TBD" H 4100 3400 50  0001 C CNN "Manufacturer PN"
+F 8 "TBD" H 4100 3400 50  0001 C CNN "Description"
 	1    4100 3400
 	-1   0    0    -1
@@
 F 4 "MSS1P4-M3/89AGICT-ND" H 6000 2700 50  0001 C CNN "Part No."
 F 5 "<a href=\"https://www.digikey.com/products/en?keywords=MSS1P4-M3/89AGICT-ND\">Link</a>" H 6000 2700 50  0001 C CNN "Link"
+F 6 "TBD" H 6000 2700 50  0001 C CNN "Manufacturer"
+F 7 "TBD" H 6000 2700 50  0001 C CNN "Manufacturer PN"
+F 8 "TBD" H 6000 2700 50  0001 C CNN "Description"
 	1    6000 2700
 	-1   0    0    -1
@@
 F 4 "MMBT2222ATPMSCT-ND" H 2050 5900 50  0001 C CNN "Part No."
 F 5 "<a href=\"https://www.digikey.com/products/en?keywords=MMBT2222ATPMSCT-ND\">Link</a>" H 2050 5900 50  0001 C CNN "Link"
-F 6 "" H 2050 5900 50  0001 C CNN "Manufacturer"
+F 6 "TBD" H 2050 5900 50  0001 C CNN "Manufacturer"
+F 7 "TBD" H 2050 5900 50  0001 C CNN "Manufacturer PN"
+F 8 "TBD" H 2050 5900 50  0001 C CNN "Description"
 	1    2050 5900
 	-1   0    0    -1
@@
 F 4 "MMBT2222ATPMSCT-ND" H 6450 3550 50  0001 C CNN "Part No."
 F 5 "<a href=\"https://www.digikey.com/products/en?keywords=MMBT2222ATPMSCT-ND\">Link</a>" H 6450 3550 50  0001 C CNN "Link"
+F 6 "TBD" H 6450 3550 50  0001 C CNN "Manufacturer"
+F 7 "TBD" H 6450 3550 50  0001 C CNN "Manufacturer PN"
+F 8 "TBD" H 6450 3550 50  0001 C CNN "Description"
 	1    6450 3550
 	-1   0    0    -1
@@
 F 4 "311-10.0KCRCT-ND" H 6350 3100 60  0001 C CNN "Part No."
 F 5 "<a href=\"https://www.digikey.com/products/en?keywords=311-10.0KCRCT-ND\">Link</a>" H 6350 3100 60  0001 C CNN "Link"
+F 6 "TBD" H 6350 3100 50  0001 C CNN "Manufacturer"
+F 7 "TBD" H 6350 3100 50  0001 C CNN "Manufacturer PN"
+F 8 "TBD" H 6350 3100 50  0001 C CNN "Description"
 	1    6350 3100
 	1    0    0    -1
@@
 F 4 "732-4984-1-ND" H 7400 5950 50  0001 C CNN "Part No."
 F 5 "<a href=\"https://www.digikey.com/products/en?keywords=732-4984-1-ND\">Link</a>" H 7400 5950 50  0001 C CNN "Link"
+F 6 "TBD" H 7400 5950 50  0001 C CNN "Manufacturer"
+F 7 "TBD" H 7400 5950 50  0001 C CNN "Manufacturer PN"
+F 8 "TBD" H 7400 5950 50  0001 C CNN "Description"
 	1    7400 5950
 	-1   0    0    1
