File: kicad/Arducon.sch (KiCad schematic (older format))
At the start: 74 parts, among them J101 To Radio, J102 DB9 Female, J103 To Antenna, J104 Conn_01x08, J105 Conn_01x08, J106 Logic Level, J107 External Power Source, J108 Controlled Power, J111 DB9_Male, J112 Conn_01x06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

Commit message: Sync
Sync of KiCad changes
Parts:
- removed D101: MSS1P2L-M3/89A, Diodes_SMD:DO-219AD, symbol Arducon-rescue:MSS1P4-M3_89A-Diode
- removed J106: Logic Level, Pin_Headers:Pin_Header_Straight_1x04, symbol Connector_Generic:Conn_01x04
- added D101: 4.3V, Diodes_SMD:SOD-123, symbol Device:D_Zener_ALT
- added J106: Wiring, Pin_Headers:Pin_Header_Straight_1x08, symbol Connector_Generic:Conn_01x08
Connections:
- net CW_KEY: now also J106.3 (Pin_3)
- net EXT_BATTERY: now also D101.1 (K), J106.8 (Pin_8)
- net GND: now also J106.1 (Pin_1)
- net PTT_LOGIC: now also J106.4 (Pin_4)
- net TONE_LOGIC: now also J106.2 (Pin_2)
- net at MOD101.24 (RAW): now also D101.2 (A)
- net AUDIO_IN renamed Audio_In
- net Audio_In: now also J106.5 (Pin_5)
- net AUDIO_OUT renamed Audio_Out
- net Audio_Out: now also J106.7 (Pin_7)
- net PTT_OUT renamed PTT_Out
- net PTT_Out: now also J106.6 (Pin_6)
Other:
- moved on the sheet: C103, Q101, R101, R102, R104, RV101, SJ102

Commit message: PCB Updates
o Added D110 to schematic and PCB to protect any connected computer from overvoltage due to an attached battery
o Added footprints for D102 and SW101 to the back side of the PCB as alternative mounting locations
o Added more stitching via to attenuator board
o Updated Gerbers, drills, and placement files
Parts:
- added D110: MSS1P2L-M3/89A, Diodes_SMD:DO-219AD, symbol Arducon-rescue:MSS1P4-M3_89A-Diode
Connections:
- net Power_In: now also D110.1 (K); no longer FB102.1
- new net: D110.2 (A), FB102.1
Other:
- moved on the sheet: SW102
Changed lines of the file:
@@
 Sheet 1 2
 Title "Arducon"
-Date "2021-05-01"
-Rev "P2.2"
+Date "2021-10-24"
+Rev "V2.5"
 Comp ""
 Comment1 ""
@@
 	0    -1   -1   0
 $EndComp
-Text GLabel 3450 2150 2    39   Output ~ 0
+Text GLabel 3850 2150 2    39   Output ~ 0
 EXT_BATTERY
 Text GLabel 11600 9950 0    39   Input ~ 0
@@
 L Arducon-rescue:Vproc-power #PWR0156
 U 1 1 5FDC95A5
-P 2750 1950
-F 0 "#PWR0156" H 2750 1800 50  0001 C CNN
-F 1 "Vproc" V 2750 2200 50  0000 C CNN
-F 2 "" H 2750 1950 50  0000 C CNN
-F 3 "" H 2750 1950 50  0000 C CNN
-	1    2750 1950
+P 3150 1950
+F 0 "#PWR0156" H 3150 1800 50  0001 C CNN
+F 1 "Vproc" V 3150 2200 50  0000 C CNN
+F 2 "" H 3150 1950 50  0000 C CNN
+F 3 "" H 3150 1950 50  0000 C CNN
+	1    3150 1950
 	0    1    1    0
 $EndComp
@@
 L Switch:SW_SPDT SW102
 U 1 1 6042734C
-P 2550 2050
-F 0 "SW102" H 2750 2050 50  0000 C CNN
-F 1 "5V/12V" H 3100 2050 50  0000 C CNN
-F 2 "Buttons_Switches_SMD:SW_SPDT_PCM12" H 2550 2050 50  0001 C CNN
-F 3 "" H 2550 2050 50  0001 C CNN
-F 4 "401-2016-1-ND" H 2550 2050 50  0001 C CNN "Digi-Key Part No."
-F 5 "<a href=\"https://www.digikey.com/products/en?keywords=401-2016-1-ND\">Link</a>" H 2550 2050 50  0001 C CNN "Link"
-F 6 "C&K" H 2550 2050 50  0001 C CNN "Manufacturer"
-F 7 "PCM12SMTR" H 2550 2050 50  0001 C CNN "Manufacturer PN"
-F 8 "SWITCH SLIDE SPDT 300MA 6V" H 2550 2050 50  0001 C CNN "Description"
-F 9 "C221841" H 2550 2050 50  0001 C CNN "LCSC Part Number"
-	1    2550 2050
+P 2950 2050
+F 0 "SW102" H 3150 2050 50  0000 C CNN
+F 1 "5V/12V" H 3500 2050 50  0000 C CNN
+F 2 "Buttons_Switches_SMD:SW_SPDT_PCM12" H 2950 2050 50  0001 C CNN
+F 3 "" H 2950 2050 50  0001 C CNN
+F 4 "401-2016-1-ND" H 2950 2050 50  0001 C CNN "Digi-Key Part No."
+F 5 "<a href=\"https://www.digikey.com/products/en?keywords=401-2016-1-ND\">Link</a>" H 2950 2050 50  0001 C CNN "Link"
+F 6 "C&K" H 2950 2050 50  0001 C CNN "Manufacturer"
+F 7 "PCM12SMTR" H 2950 2050 50  0001 C CNN "Manufacturer PN"
+F 8 "SWITCH SLIDE SPDT 300MA 6V" H 2950 2050 50  0001 C CNN "Description"
+F 9 "C221841" H 2950 2050 50  0001 C CNN "LCSC Part Number"
+	1    2950 2050
 	1    0    0    -1
 $EndComp
@@
 	2000 1650 4100 1650
 Connection ~ 4100 1650
-Wire Wire Line
-	2300 2400 2300 2050
-Wire Wire Line
-	2300 2050 2350 2050
-Text GLabel 2350 2400 2    39   Output ~ 0
+Text GLabel 3350 2400 2    39   Output ~ 0
 Power_In
-Wire Wire Line
-	2350 2400 2300 2400
 Text GLabel 2500 5650 0    39   Input ~ 0
 Power_In
@@
 	1900 2400 1650 2400
 Wire Wire Line
-	2100 2400 2300 2400
-Connection ~ 2300 2400
-Wire Wire Line
 	1900 2200 1650 2200
 Wire Wire Line
@@
 Connection ~ 13800 3650
 Wire Wire Line
-	3450 2150 2750 2150
+	3850 2150 3150 2150
 $Comp
 L Device:D_Zener_ALT D101
@@
 Wire Wire Line
 	2000 1500 2000 1650
-Wire Bus Line
-	6150 4000 6150 6700
 Connection ~ 2000 1650
 Text GLabel 1450 4350 2    39   Input ~ 0
 Audio_Out
+$Comp
+L Arducon-rescue:MSS1P4-M3_89A-Diode D110
+U 1 1 6176C6A6
+P 2500 2400
+F 0 "D110" H 2500 2500 50  0000 C CNN
+F 1 "MSS1P2L-M3/89A" H 2650 2650 50  0001 C CNN
+F 2 "Diodes_SMD:DO-219AD" H 2500 2225 50  0001 C CNN
+F 3 "" H 2500 2400 50  0001 C CNN
+F 4 "MSS1P2L-M3/89AGICT-ND" H 2500 2400 50  0001 C CNN "Digi-Key Part No."
+F 5 "<a href=\"https://www.digikey.com/products/en?keywords=MSS1P2L-M3/89AGICT-ND\">Link</a>" H 2500 2400 50  0001 C CNN "Link"
+F 6 "Vishay General Semiconductor" H 2500 2400 50  0001 C CNN "Manufacturer"
+F 7 "MSS1P2L-M3/89A" H 2500 2400 50  0001 C CNN "Manufacturer PN"
+F 8 "DIODE SCHOTTKY 20V 1A MICROSMP" H 2500 2400 50  0001 C CNN "Description"
+F 9 "C506621" H 2500 2400 50  0001 C CNN "LCSC Part Number"
+	1    2500 2400
+	-1   0    0    -1
+$EndComp
+Wire Wire Line
+	2100 2400 2350 2400
+Wire Wire Line
+	2650 2400 2700 2400
+Wire Wire Line
+	2700 2400 2700 2050
+Wire Wire Line
+	2700 2050 2750 2050
+Wire Wire Line
+	3350 2400 2700 2400
+Wire Bus Line
+	6150 4000 6150 6700
+Connection ~ 2700 2400
 $EndSCHEMATC
