File: kicad/Non-PCB-Parts.sch (KiCad schematic (older format))
At the start: 1 part

Commit message: Schematic Update
Changed schematic and PCB design to support two different RTC devices: DS3132 and RV-8803-C7. Only one RTC option should be populated.
Parts:
- PCB201: Digi-Key Part No. (none) -> np; Part No. np -> (none)
Changed lines of the file:
@@
 F 2 "Oddities:Dummy_Empty" H 3990 2510 50  0001 C CNN
 F 3 "" H 3990 2510 50  0001 C CNN
-F 4 "np" H 3150 2350 50  0001 C CNN "Part No."
+F 4 "np" H 3150 2350 50  0001 C CNN "Digi-Key Part No."
 F 5 "np" H 3150 2350 50  0001 C CNN "Link"
 	1    3150 2350
